File: docs/reverse_engineering/nRF52840_Microcontroller/schematic/schematic.kicad_sch (KiCad schematic)
At the start: 1 part, among them U1 nRF52840

Commit message: Release commit
Parts:
- added D1, D10, D11, D12, D13, D14, D15, D16, D17, D18, D19, D2, D20, D21, D22, D23, D24, D25, D26, D27, D28, D29, D3, D30, D31, D32, D33, D34, D35, D36, D37, D38, D39, D4, D40, D41, D42, D43, D44, D45, D46, D47, D48, D49, D5, D50, D51, D52, D6, D7, D8, D9: D_Small, symbol Device:D_Small
- added MX1: Y, PCM_marbastlib-mx:SW_MX_1u, symbol PCM_marbastlib-mx:MX_SW_solder
- added MX10: L, PCM_marbastlib-mx:SW_MX_1u, symbol PCM_marbastlib-mx:MX_SW_solder
- added MX11: ;, PCM_marbastlib-mx:SW_MX_1u, symbol PCM_marbastlib-mx:MX_SW_solder
- added MX12: ', PCM_marbastlib-mx:SW_MX_1u, symbol PCM_marbastlib-mx:MX_SW_solder
- added MX13: N, PCM_marbastlib-mx:SW_MX_1u, symbol PCM_marbastlib-mx:MX_SW_solder
- added MX14: M, PCM_marbastlib-mx:SW_MX_1u, symbol PCM_marbastlib-mx:MX_SW_solder
- added MX15: <, PCM_marbastlib-mx:SW_MX_1u, symbol PCM_marbastlib-mx:MX_SW_solder
- added MX16: >, PCM_marbastlib-mx:SW_MX_1u, symbol PCM_marbastlib-mx:MX_SW_solder
- added MX17: /, PCM_marbastlib-mx:SW_MX_1u, symbol PCM_marbastlib-mx:MX_SW_solder
- added MX18: FN, PCM_marbastlib-mx:SW_MX_1u, symbol PCM_marbastlib-mx:MX_SW_solder
- added MX19: [, PCM_marbastlib-mx:SW_MX_1u, symbol PCM_marbastlib-mx:MX_SW_solder
- added MX2: U, PCM_marbastlib-mx:SW_MX_1u, symbol PCM_marbastlib-mx:MX_SW_solder
- added MX20: ], PCM_marbastlib-mx:SW_MX_1u, symbol PCM_marbastlib-mx:MX_SW_solder
- added MX21: SYS, PCM_marbastlib-mx:SW_MX_1u, symbol PCM_marbastlib-mx:MX_SW_solder
- added MX22, MX50: CTRL, PCM_marbastlib-mx:SW_MX_1u, symbol PCM_marbastlib-mx:MX_SW_solder
- added MX23: ENTER, PCM_marbastlib-mx:SW_MX_1u, symbol PCM_marbastlib-mx:MX_SW_solder
- added MX24: BACKSPACE, PCM_marbastlib-mx:SW_MX_1u, symbol PCM_marbastlib-mx:MX_SW_solder
- added MX25, MX51: DOT, PCM_marbastlib-mx:SW_MX_1u, symbol PCM_marbastlib-mx:MX_SW_solder
- added MX26, MX49: ALT, PCM_marbastlib-mx:SW_MX_1u, symbol PCM_marbastlib-mx:MX_SW_solder
- added MX27: ESC, PCM_marbastlib-mx:SW_MX_1u, symbol PCM_marbastlib-mx:MX_SW_solder
- added MX28: Q, PCM_marbastlib-mx:SW_MX_1u, symbol PCM_marbastlib-mx:MX_SW_solder
- added MX29: W, PCM_marbastlib-mx:SW_MX_1u, symbol PCM_marbastlib-mx:MX_SW_solder
- added MX3: I, PCM_marbastlib-mx:SW_MX_1u, symbol PCM_marbastlib-mx:MX_SW_solder
- added MX30: TAB, PCM_marbastlib-mx:SW_MX_1u, symbol PCM_marbastlib-mx:MX_SW_solder
- added MX31: A, PCM_marbastlib-mx:SW_MX_1u, symbol PCM_marbastlib-mx:MX_SW_solder
- added MX32: S, PCM_marbastlib-mx:SW_MX_1u, symbol PCM_marbastlib-mx:MX_SW_solder
- added MX33: FUN, PCM_marbastlib-mx:SW_MX_1u, symbol PCM_marbastlib-mx:MX_SW_solder
- added MX34: Z, PCM_marbastlib-mx:SW_MX_1u, symbol PCM_marbastlib-mx:MX_SW_solder
- added MX35: X, PCM_marbastlib-mx:SW_MX_1u, symbol PCM_marbastlib-mx:MX_SW_solder
- added MX36: E, PCM_marbastlib-mx:SW_MX_1u, symbol PCM_marbastlib-mx:MX_SW_solder
- added MX37: CAPSLOCK, PCM_marbastlib-mx:SW_MX_1u, symbol PCM_marbastlib-mx:MX_SW_solder
- added MX38: FNSW, PCM_marbastlib-mx:SW_MX_1u, symbol PCM_marbastlib-mx:MX_SW_solder
- added MX39: D, PCM_marbastlib-mx:SW_MX_1u, symbol PCM_marbastlib-mx:MX_SW_solder
- added MX4: O, PCM_marbastlib-mx:SW_MX_1u, symbol PCM_marbastlib-mx:MX_SW_solder
- added MX40: C, PCM_marbastlib-mx:SW_MX_1u, symbol PCM_marbastlib-mx:MX_SW_solder
- added MX41: R, PCM_marbastlib-mx:SW_MX_1u, symbol PCM_marbastlib-mx:MX_SW_solder
- added MX42: T, PCM_marbastlib-mx:SW_MX_1u, symbol PCM_marbastlib-mx:MX_SW_solder
- added MX43: F, PCM_marbastlib-mx:SW_MX_1u, symbol PCM_marbastlib-mx:MX_SW_solder
- added MX44: G, PCM_marbastlib-mx:SW_MX_1u, symbol PCM_marbastlib-mx:MX_SW_solder
- added MX45: V, PCM_marbastlib-mx:SW_MX_1u, symbol PCM_marbastlib-mx:MX_SW_solder
- added MX46: B, PCM_marbastlib-mx:SW_MX_1u, symbol PCM_marbastlib-mx:MX_SW_solder
- added MX47: SHIFT, PCM_marbastlib-mx:SW_MX_1u, symbol PCM_marbastlib-mx:MX_SW_solder
- added MX48: SPACE, PCM_marbastlib-mx:SW_MX_1u, symbol PCM_marbastlib-mx:MX_SW_solder
- added MX5: P, PCM_marbastlib-mx:SW_MX_1u, symbol PCM_marbastlib-mx:MX_SW_solder
- added MX52: DEL, PCM_marbastlib-mx:SW_MX_1u, symbol PCM_marbastlib-mx:MX_SW_solder
- added MX6: \, PCM_marbastlib-mx:SW_MX_1u, symbol PCM_marbastlib-mx:MX_SW_solder
- added MX7: H, PCM_marbastlib-mx:SW_MX_1u, symbol PCM_marbastlib-mx:MX_SW_solder
- added MX8: J, PCM_marbastlib-mx:SW_MX_1u, symbol PCM_marbastlib-mx:MX_SW_solder
- added MX9: K, PCM_marbastlib-mx:SW_MX_1u, symbol PCM_marbastlib-mx:MX_SW_solder
Connections:
- new net: D47.1 (K), MX47.2
- new net: D25.1 (K), MX25.2
- new net: D33.1 (K), MX33.2
- new net: D22.1 (K), MX22.2
- new net: D48.1 (K), MX48.2
- new net: D28.1 (K), MX28.2
- new net: D9.1 (K), MX12.2
- new net: D2.1 (K), MX2.2
- new net: D15.1 (K), MX18.2
- new net: D46.1 (K), MX46.2
- new net: D18.1 (K), MX15.2
- new net: D32.1 (K), MX32.2
- new net: D36.1 (K), MX36.2
- new net: D35.1 (K), MX35.2
- new net: D21.1 (K), MX21.2
- new net: D8.1 (K), MX11.2
- new net: D27.1 (K), MX27.2
- new net: D44.1 (K), MX44.2
- new net: D34.1 (K), MX34.2
- new net: D29.1 (K), MX29.2
- new net: D16.1 (K), MX13.2
- new net: D45.1 (K), MX45.2
- new net: D31.1 (K), MX31.2
- new net: D10.1 (K), MX7.2
- new net: D49.1 (K), MX49.2
- new net: D52.1 (K), MX52.2
- new net: D43.1 (K), MX43.2
- new net: D23.1 (K), MX23.2
- new net: D19.1 (K), MX20.2
- new net: D41.1 (K), MX41.2
- new net: D17.1 (K), MX14.2
- new net: D50.1 (K), MX50.2
- new net: D20.1 (K), MX19.2
- new net: D1.1 (K), MX1.2
- new net: D3.1 (K), MX3.2
- new net: D38.1 (K), MX38.2
- new net: D7.1 (K), MX10.2
- new net: D51.1 (K), MX51.2
- new net: D13.1 (K), MX16.2
- new net: D40.1 (K), MX40.2
- new net: D24.1 (K), MX24.2
- new net: D5.1 (K), MX5.2
- new net: D11.1 (K), MX8.2
- new net: D12.1 (K), MX9.2
- new net: D14.1 (K), MX17.2
- new net: D42.1 (K), MX42.2
- new net: D37.1 (K), MX37.2
- new net: D4.1 (K), MX4.2
- new net: D6.1 (K), MX6.2
- new net: D30.1 (K), MX30.2
- new net: D26.1 (K), MX26.2
- new net: D39.1 (K), MX39.2
- new net P0.02: MX13.1, MX14.1, MX15.1, MX16.1, MX17.1, MX18.1, MX23.1, MX25.1, MX33.1, MX34.1, MX35.1, MX40.1, MX45.1, MX46.1, MX48.1, MX51.1
- new net P0.03: MX19.1, MX20.1, MX37.1, MX38.1
- new net P0.28: MX10.1, MX11.1, MX12.1, MX22.1, MX26.1, MX30.1, MX31.1, MX32.1, MX39.1, MX43.1, MX44.1, MX49.1, MX50.1, MX7.1, MX8.1, MX9.1
- new net P0.29: MX1.1, MX2.1, MX21.1, MX24.1, MX27.1, MX28.1, MX29.1, MX3.1, MX36.1, MX4.1, MX41.1, MX42.1, MX47.1, MX5.1, MX52.1, MX6.1
- new net P0.30: D21.2 (A), D22.2 (A), D23.2 (A), D48.2 (A), D50.2 (A), D52.2 (A)
- new net P0.31: D24.2 (A), D25.2 (A), D26.2 (A), D47.2 (A), D49.2 (A), D51.2 (A)
- new net P1.10: D1.2 (A), D10.2 (A), D16.2 (A), D42.2 (A), D44.2 (A), D46.2 (A)
- new net P1.11: D11.2 (A), D17.2 (A), D2.2 (A), D41.2 (A), D43.2 (A), D45.2 (A)
- new net P1.12: D12.2 (A), D18.2 (A), D20.2 (A), D3.2 (A), D36.2 (A), D38.2 (A), D39.2 (A), D40.2 (A)
- new net P1.13: D13.2 (A), D19.2 (A), D29.2 (A), D32.2 (A), D35.2 (A), D37.2 (A), D4.2 (A), D7.2 (A)
- new net P1.14: D14.2 (A), D28.2 (A), D31.2 (A), D34.2 (A), D5.2 (A), D8.2 (A)
- new net P1.15: D15.2 (A), D27.2 (A), D30.2 (A), D33.2 (A), D6.2 (A), D9.2 (A)
Other:
- moved on the sheet: U1
